Commit message: 抓杯子阶段，真机部署成功版本

File: fr5_description/urdf/fr5v6.urdf (robot description, URDF)
Before this commit: robot fr5v6, 11 links, 10 joints
Links:
- link finger_link1: mass 0.0589543896992846 -> 1; geometry collision box size=0.01 0.08 0.03; visual box size=0.01 0.08 0.03
- link finger_link2: mass 0.0589543896992846 -> 1; geometry collision box size=0.01 0.08 0.03; visual box size=0.01 0.08 0.03
Joints:
- joint fj1: limit lower=0 upper=0.04 effort=40 velocity=1 -> lower=0 upper=0.04 effort=200 velocity=0.0001
- joint fj2: limit lower=0 upper=0.04 effort=40 velocity=1 -> lower=0 upper=0.04 effort=200 velocity=0.0001

Commit message: pick_and_place仿真成功版本

File: fr5_description/urdf/fr5v6.urdf (robot description, URDF)
Before this commit: robot fr5v6, 11 links, 10 joints
Joints:
- joint fj1: limit lower=0 upper=0.04 effort=200 velocity=0.0001 -> lower=-0.05 upper=0.04 effort=20 velocity=0.1
- joint fj2: limit lower=0 upper=0.04 effort=200 velocity=0.0001 -> lower=-0.05 upper=0.04 effort=20 velocity=0.1

Commit message: 微调urdf文件

File: fr5_description/urdf/fr5v6.urdf (robot description, URDF)
Before this commit: robot fr5v6, 11 links, 10 joints
Joints:
- joint fj1: limit lower=-0.05 upper=0.04 effort=20 velocity=0.1 -> lower=-0.1 upper=0.1 effort=20 velocity=0.1
- joint fj2: limit lower=-0.05 upper=0.04 effort=20 velocity=0.1 -> lower=-0.10 upper=0.10 effort=20 velocity=0.1; origin xyz=-0.0425 0.0087157 -0.0015 rpy=1.5708 0 3.1416 -> xyz=-0.0425 0.0 -0.0 rpy=1.5708 0 3.1416

Commit message: 长序列学习，使用对齐专家模型与学习模型输出的方法，可以成功训练

File: fr5_description/urdf/fr5v6.urdf (robot description, URDF)
Before this commit: robot fr5v6, 11 links, 10 joints
Joints:
- joint fj1: limit lower=-0.05 upper=0.04 effort=20 velocity=0.1 -> lower=-0.1 upper=0.1 effort=20 velocity=0.1
- joint fj2: limit lower=-0.05 upper=0.04 effort=20 velocity=0.1 -> lower=-0.10 upper=0.10 effort=20 velocity=0.1; origin xyz=-0.0425 0.0087157 -0.0015 rpy=1.5708 0 3.1416 -> xyz=-0.0425 0.0087157 0. rpy=1.5708 0 3.1416
